File: eagle/atmega_midi_SP0256-AL2.sch (EAGLE design)
At the start: 38 parts, among them IC1 TL072P, U1 ATMEGA328P_PDIP

Commit message: mostly there with sp chip
Parts:
- removed IC1: TL072P, linear:TL072P
- removed OK1: 6N138, optocoupler:6N138
- added C13: 1uF, rcl:CPOL-USB45181A
- added C14, C15: 27pF, rcl:C-US025-040X050
- added Q2: (no value), crystal:CRYSTALHC49S
- added U2: ATMEGA328P_PDIP, SparkFun-DigitalIC:ATMEGA328P_PDIP
- added U4: TL072P, linear:TL072P
- C6: value 100n -> 3n
- R4: value 1k -> 10k
- U1: value ATMEGA328P_PDIP -> 6N138; device SparkFun-DigitalIC:ATMEGA328P_PDIP -> optocoupler:6N138
- renumbered U$5 to U3
Connections:
- new net N$15: U2.PD3(INT1), U3.SE
- new net N$17: C13.+, U3.DIGITALOUT
- new net N$19: U2.PC0(ADC0), U3.A1
- new net N$21: U2.PC1(ADC1), U3.A2
- new net N$23: U2.PC2(ADC2), U3.A3
- new net N$24: U2.PC3(ADC3), U3.A4
- new net N$25: U2.PC4(ADC4/SDA), U3.A5
- new net N$26: U2.PC5(ADC5/SCL), U3.A6
- new net N$27: U2.PD2(INT0), U3.!ALD
- new net N$28: U2.PB4(MISO), U3.!LRQ
- new net N$32: C13.-, R4.1
- new net N$38: C14.1, Q2.1, U3.OSC2
- new net N$39: C15.1, Q2.2, U3.OSC1
- net +12V: now also U4P.V+; no longer IC1P.V+
- net +5V: now also U2.VCC, U3.!RESET, U3.!SBYRESET, U3.VD1, U3.VDD; no longer OK1.VCC
- net -12V: now also U4P.V-; no longer IC1P.V-
- net GND: now also C14.2, C15.2, C6.2, U3.TEST, U3.VSS
- net N$10: now also U4B.-IN; no longer IC1B.-IN
- net N$12: now also U4A.-IN, U4A.OUT; no longer IC1A.-IN, IC1A.OUT
- net N$16: now also U4B.OUT; no longer IC1B.OUT
- net N$20: now also U2.PD6(AIN0); no longer U1.PD6(AIN0)
- net N$22: now also U2.PD4(XCK/T0), U4B.+IN; no longer IC1B.+IN, U1.PD4(XCK/T0)
- net N$29: now also U1.GND, U2.GND@1, U2.GND@2; no longer OK1.GND, U1.GND@1, U1.GND@2
- net N$3: now also U1.C; no longer OK1.C
- net N$30: now also U1.VO, U2.PD0(RXD); no longer OK1.VO, U1.PD0(RXD)
- net N$4: now also U2.PB6(XTAL1/TOSC1); no longer U1.PB6(XTAL1/TOSC1)
- net N$43: now also U2.PC6(/RESET); no longer U1.PC6(/RESET)
- net N$5: now also U2.PB7(XTAL2/TOSC2); no longer U1.PB7(XTAL2/TOSC2)
- net N$6: now also C6.1, R4.2, U4A.+IN; no longer IC1A.+IN
- net N$7: now also U1.A; no longer OK1.A
Other:
- moved on the sheet: AMT, C6, OUTPUT, R10, R25, R4, VEL_LED

Commit message: layout adjusting
Parts:
- added RESET2: LSP11, solpad:LSP11
- RESET: value 22-23-2021 -> LSP11; device con-molex:22-23-2021 -> solpad:LSP11
- renumbered U$4 to MIDI_IN
Connections:
- net GND: now also MIDI_ING$2.MT, MIDI_ING$3.MT, MIDI_ING$4.MT, MIDI_ING$5.MT
- net N$15: now also U2.PB4(MISO), U3.!ALD; no longer U2.PD3(INT1), U3.SE
- net N$27: now also U2.PB5(SCK), U3.SE; no longer U2.PD2(INT0), U3.!ALD
- net N$28: now also U2.PB1(OC1A); no longer U2.PB4(MISO)
- net N$29: now also RESET2.MP; no longer RESET-2.S
- net N$43: now also RESET.MP; no longer RESET-1.S
Other:
- moved on the sheet: U2

Commit message: 93pct auto
Connections:
- removed net N$1: C4.2, C7.1
- net GND: now also C4.2, C7.1, GATE.RING, OUTPUT.RING, R13.2, RESET2.MP, U1.GND
- net N$28: now also U2.PB3(MOSI/OC2); no longer U2.PB1(OC1A)
- net N$29: no longer GATE.RING, OUTPUT.RING, R13.2, RESET2.MP, U1.GND

Commit message: routed
Parts:
- added C16: 100n, rcl:C-US025-030X050
- C10, C12, C3, C7, C8: device rcl:C-US050-024X044 -> rcl:C-US025-030X050
Connections:
- removed net N$29: C1.1, C10.1, C11.-, C12.2, C2.1, C3.2, C5.-, C8.2, C9.+, PWR1.GND, U2.GND@1, U2.GND@2
- net +5V: now also C16.1
- net GND: now also C1.1, C10.1, C11.-, C12.2, C16.2, C2.1, C3.2, C5.-, C8.2, C9.+, PWR1.GND, U2.GND@1, U2.GND@2
Other:
- moved on the sheet: AMT, C10, C6, C9, MIDI_ING$1, OUTPUT, R10, U$1, U4A
